Commit message: Readd topics_ns:=camera  argument

File: realsense2_description/urdf/_d435.urdf.xacro (robot description, xacro)
@@ -11,5 +11,5 @@
   <xacro:include filename="$(find realsense2_description)/urdf/_materials.urdf.xacro" />
   <xacro:include filename="$(find realsense2_description)/urdf/_usb_plug.urdf.xacro" />
-  <xacro:macro name="sensor_d435" params="parent *origin name:=camera use_nominal_extrinsics:=false add_plug:=false use_mesh:=true publish_pointcloud:=true">
+  <xacro:macro name="sensor_d435" params="parent *origin name:=camera topics_ns:=camera use_nominal_extrinsics:=false add_plug:=false use_mesh:=true publish_pointcloud:=true">
     <xacro:property name="M_PI" value="3.1415926535897931" />
     <!-- The following values are approximate, and the camera node

Commit message: fix d435 inertia parameters

File: realsense2_description/urdf/_d435.urdf.xacro (robot description, xacro)
@@ -24,4 +24,6 @@
     <xacro:property name="d435_cam_depth" value="0.02505"/>
     <xacro:property name="d435_cam_mount_from_center_offset" value="0.0149"/>
+    <!-- mass of D435 camera -->
+    <xacro:property name="d435_cam_mass" value="0.072"/>
     <!-- glass cover is 0.1 mm inwards from front aluminium plate -->
     <xacro:property name="d435_glass_to_front" value="0.1e-3"/>
@@ -75,7 +77,9 @@
       <inertial>
         <!-- The following are not reliable values, and should not be used for modeling -->
-        <mass value="0.072" />
-        <origin xyz="0 0 0" />
-        <inertia ixx="0.003881243" ixy="0.0" ixz="0.0" iyy="0.000498940" iyz="0.0" izz="0.003879257" />
+        <mass value="${d435_cam_mass}" />
+        <origin xyz="${-d435_mesh_x_offset} ${-d435_cam_depth_py} 0" />
+        <inertia ixx="${(d435_cam_mass * (d435_cam_height * d435_cam_height + d435_cam_width * d435_cam_width)) / 12}" ixy="0.0" ixz="0.0"
+                 iyy="${(d435_cam_mass * (d435_cam_height * d435_cam_height + d435_cam_depth * d435_cam_depth)) / 12}" iyz="0.0"
+                 izz="${(d435_cam_mass * (d435_cam_width * d435_cam_width + d435_cam_depth * d435_cam_depth)) / 12}" />
       </inertial>
     </link>

Commit message: Externalize gazebo simulation xacro

File: realsense2_description/urdf/_d435.urdf.xacro (robot description, xacro)
@@ -8,5 +8,5 @@
 <robot name="sensor_d435" xmlns:xacro="http://ros.org/wiki/xacro">
   <!-- Includes -->
-  <xacro:include filename="$(find realsense2_description)/urdf/_d435.gazebo.xacro"/>
+  <xacro:include filename="$(find realsense_simulation)/urdf/_d435.gazebo.xacro"/>
   <xacro:include filename="$(find realsense2_description)/urdf/_usb_plug.urdf.xacro" />
   <xacro:macro name="sensor_d435" params="parent *origin name:=camera topics_ns:=camera use_nominal_extrinsics:=false add_plug:=false use_mesh:=true publish_pointcloud:=true">

File: realsense2_description/urdf/_d455.urdf.xacro (robot description, xacro)
@@ -8,5 +8,5 @@
 <robot name="sensor_d455" xmlns:xacro="http://ros.org/wiki/xacro">
   <!-- Includes -->
-  <xacro:include filename="$(find realsense2_description)/urdf/_d455.gazebo.xacro"/>
+  <xacro:include filename="$(find realsense_simulation)/urdf/_d455.gazebo.xacro"/>
   <xacro:include filename="$(find realsense2_description)/urdf/_usb_plug.urdf.xacro" />
   <xacro:macro name="sensor_d455" params="parent *origin name:=camera topics_ns:=camera use_nominal_extrinsics:=false add_plug:=false use_mesh:=true publish_pointcloud:=true">

File: realsense2_description/urdf/_l515.urdf.xacro (robot description, xacro)
@@ -10,5 +10,6 @@
   <xacro:include filename="$(find realsense2_description)/urdf/_materials.urdf.xacro" />
   <xacro:include filename="$(find realsense2_description)/urdf/_usb_plug.urdf.xacro" /> <!-- this specific plug does not apply to L515 -->
-  <xacro:macro name="sensor_l515" params="parent *origin name:=camera use_nominal_extrinsics:=false add_plug:=false use_mesh:=true">
+  <xacro:include filename="$(find realsense_simulation)/urdf/_l515.gazebo.xacro" />
+  <xacro:macro name="sensor_l515" params="parent *origin name:=camera use_nominal_extrinsics:=false add_plug:=false use_mesh:=true topics_ns:=camera">
     <xacro:property name="M_PI" value="3.1415926535897931" />
     <!-- The following values are approximate, and the camera node
@@ -172,4 +173,6 @@
       </xacro:usb_plug>
     </xacro:if>
+    <!-- Realsense Gazebo Plugin -->
+    <xacro:gazebo_l515 camera_name="${name}" reference_link="${name}_link" topics_ns="${topics_ns}" depth_optical_frame="${name}_depth_optical_frame" color_optical_frame="${name}_color_optical_frame" infrared_optical_frame="${name}_infra_optical_frame"/>
   </xacro:macro>
 </robot>

File: realsense2_description/urdf/_t265.urdf.xacro (robot description, xacro)
@@ -8,5 +8,5 @@
 <robot name="sensor_t265" xmlns:xacro="http://ros.org/wiki/xacro">
   <!--File includes-->
-  <xacro:include filename="$(find realsense2_description)/urdf/_t265.gazebo.xacro"/>
+  <xacro:include filename="$(find realsense_simulation)/urdf/_t265.gazebo.xacro"/>
   <xacro:macro name="sensor_t265" params="parent name:=camera topics_ns:=camera *origin">
     <xacro:property name="M_PI" value="3.1415926535897931" />

Commit message: Fix dae mesh + replace by a simplified mesh for simulation

File: realsense2_description/urdf/_d435.urdf.xacro (robot description, xacro)
@@ -67,6 +67,7 @@
           <origin xyz="${d435_zero_depth_to_glass + d435_glass_to_front} ${-d435_cam_depth_py} 0" rpy="${M_PI/2} 0 ${M_PI/2}"/>
           <geometry>
-            <mesh filename="file://$(find realsense2_description)/meshes/d435.dae" />
+            <mesh filename="file://$(find realsense2_description)/meshes/d435_simplified.stl" />
           </geometry>
+          <material name="aluminum"/>
         </xacro:if>
         <xacro:unless value="${use_mesh}">
@@ -85,8 +86,7 @@
       </collision>
       <inertial>
-        <!-- The following are not reliable values, and should not be used for modeling -->
-        <mass value="0.072" />
-        <origin xyz="0 0 0" />
-        <inertia ixx="0.003881243" ixy="0.0" ixz="0.0" iyy="0.000498940" iyz="0.0" izz="0.003879257" />
+        <mass value="0.04475" />
+        <origin xyz="0.0019 0.00025 0.01244" />
+        <inertia ixx="0.00003" ixy="0.0" ixz="0.0" iyy="0.00003" iyz="0.0" izz="0.00003" />
       </inertial>
     </link>

Commit message: Change use mesh to false by default and replace the box by the simplified mesh

File: realsense2_description/urdf/_d435.urdf.xacro (robot description, xacro)
@@ -24,5 +24,5 @@
   <xacro:include filename="$(find realsense2_description)/urdf/_usb_plug.urdf.xacro" />
   <xacro:include filename="$(find realsense_simulation)/urdf/_d435.gazebo.xacro" />
-  <xacro:macro name="sensor_d435" params="parent *origin name:=camera use_nominal_extrinsics:=false add_plug:=false use_mesh:=true topics_ns:=camera publish_pointcloud:=true">
+  <xacro:macro name="sensor_d435" params="parent *origin name:=camera use_nominal_extrinsics:=false add_plug:=false use_mesh:=false topics_ns:=camera publish_pointcloud:=true">
     <xacro:property name="M_PI" value="3.1415926535897931" />
     <!-- The following values are approximate, and the camera node
@@ -67,5 +67,5 @@
           <origin xyz="${d435_zero_depth_to_glass + d435_glass_to_front} ${-d435_cam_depth_py} 0" rpy="${M_PI/2} 0 ${M_PI/2}"/>
           <geometry>
-            <mesh filename="file://$(find realsense2_description)/meshes/d435_simplified.stl" />
+            <mesh filename="file://$(find realsense2_description)/meshes/d435.dae" />
           </geometry>
           <material name="aluminum"/>
@@ -74,5 +74,5 @@
           <origin xyz="0 ${-d435_cam_depth_py} 0" rpy="0 0 0"/>
           <geometry>
-            <box size="${d435_cam_depth} ${d435_cam_width} ${d435_cam_height}"/>
+            <mesh filename="file://$(find realsense2_description)/meshes/d435_simplified.stl" />
           </geometry>
           <material name="aluminum"/>

Commit message: Remove material

File: realsense2_description/urdf/_d435.urdf.xacro (robot description, xacro)
@@ -69,5 +69,4 @@
             <mesh filename="file://$(find realsense2_description)/meshes/d435.dae" />
           </geometry>
-          <material name="aluminum"/>
         </xacro:if>
         <xacro:unless value="${use_mesh}">

Commit message: Fix position + collision + inertia of d435

File: realsense2_description/urdf/_d435.urdf.xacro (robot description, xacro)
@@ -71,5 +71,5 @@
         </xacro:if>
         <xacro:unless value="${use_mesh}">
-          <origin xyz="0 ${-d435_cam_depth_py} 0" rpy="0 0 0"/>
+          <origin xyz="${d435_zero_depth_to_glass + d435_glass_to_front} ${-d435_cam_depth_py} 0" rpy="${M_PI/2} 0 ${M_PI/2}"/>
           <geometry>
             <mesh filename="file://$(find realsense2_description)/meshes/d435_simplified.stl" />
@@ -79,5 +79,5 @@
       </visual>
       <collision>
-        <origin xyz="0 ${-d435_cam_depth_py} 0" rpy="0 0 0"/>
+        <origin xyz="${-d435_cam_depth/2 + d435_zero_depth_to_glass} ${-d435_cam_depth_py} 0" rpy="0 0 0"/>
         <geometry>
           <box size="${d435_cam_depth} ${d435_cam_width} ${d435_cam_height}"/>
@@ -85,7 +85,7 @@
       </collision>
       <inertial>
-        <mass value="0.04475" />
-        <origin xyz="0.0019 0.00025 0.01244" />
-        <inertia ixx="0.00003" ixy="0.0" ixz="0.0" iyy="0.00003" iyz="0.0" izz="0.00003" />
+        <mass value="0.075" />
+        <origin xyz="0.0019 -0.01244 0.00025 " />
+        <inertia ixx="0.00005" ixy="0.0" ixz="0.0" iyy="0.00001" iyz="0.0" izz="0.00005" />
       </inertial>
     </link>

Commit message: Fix origin of inertia matrix

File: realsense2_description/urdf/_d435.urdf.xacro (robot description, xacro)
@@ -86,5 +86,5 @@
       <inertial>
         <mass value="0.075" />
-        <origin xyz="0.0019 -0.01244 0.00025 " />
+        <origin xyz="-0.0087 -0.01725  -0.00006" />
         <inertia ixx="0.00005" ixy="0.0" ixz="0.0" iyy="0.00001" iyz="0.0" izz="0.00005" />
       </inertial>
